File: C64 Pi1541-III Module/C64 Pi1541-III Module.kicad_pcb (KiCad board)
At the start: 2 copper layers, 100 x 100 mm, 38 parts, among them J1 DC IN, J2 C64_IEC, J3 C64_IEC, J4 USB_C_Receptacle_USB2.0, J8 Module_Panel, M1 Mounting, M2 Mounting, M3 Mounting, M4 Mounting, Q1 DMG2302U, Q2 DMG2302U, Q3 DMG2302U, Q4 DMG2302U, U1 7406

Commit message: Add files + SMD panel
Parts:
- moved J8 8.03 mm to (120.2, 132.9)
- moved R6 3.97 mm to (114.9, 129.4)
Routing:
- net SW3_DOWN: track 89.3 -> 75.5 mm
- net SW5_INSERT: track 63.6 -> 49.8 mm, vias 1 -> 3
- net SW4_BACK: track 91.0 -> 77.3 mm, vias 1 -> 3
- net SW2_UP: track 84.6 -> 72.2 mm
- net SW1_ENTER: track 80.5 -> 70.6 mm
- net I2C_SDA: track 91.4 -> 82.7 mm
- net I2C_SCL: track 88.2 -> 80.1 mm
- net +3V3: track 214.7 -> 208.3 mm, vias 7 -> 8
- net LED_ACT: track 14.5 -> 9.02 mm
- net RPI_LED: track 57.5 -> 52.5 mm
- net LED_PWR: track 8.01 -> 4.04 mm
